File: NodePilot.kicad_sch (KiCad schematic)
At the start: 24 parts, among them K1 SRD-05VDC-SL-C, Q1 2N3904, Q3 2N3904, Q4 2N3904, T1 1:1 600R, T2 1:1 600R, U2 PC817

Commit message: change of resistor
Parts:
- R2: value 330 ohm -> 220 ohm
Changed lines of the file:
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@@
 			)
 		)
-		(property "Value" "330 ohm"
+		(property "Value" "220 ohm"
 			(at 123.19 113.0299 0)
 			(effects
