File: NodePilot.kicad_sch (KiCad schematic)
At the start: 28 parts, among them K1 SRD-05VDC-SL-C, Q3 2N3904, Q4 2N3904, T1 1:1 600R, T2 1:1 600R, U2 PC817

Commit message: version 4.2
Parts:
- removed D3: 1N5817, Diode_THT:D_DO-41_SOD81_P10.16mm_Horizontal, symbol Diode:1N5817
- added D3: 1N4148, Diode_THT:D_DO-35_SOD27_P7.62mm_Horizontal, symbol Diode:1N4148
- added R5: 2.2k ohm, symbol Device:R_US
- R10: value 10k ohm -> 2.2k ohm
- R11: value 330 ohm -> 220 ohm
- R3: value 10k ohm -> 330 ohm
Connections:
- net +5Vc: now also D3.1 (K); no longer R3.2
- net AGND1: now also R3.2
- net PTT: now also R5.2; no longer K1.3
- net at C5.2, C9.2, K1.2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: now also D3.2 (A)
- new net: K1.3, R5.1

Commit message: version v4.2 stable
Parts:
- removed D2: R_LED, symbol Device:LED
- removed R2: 1k ohm, symbol Device:R_US
- added RV3: 10k, symbol Device:R_Potentiometer_US
Connections:
- net RIGAF: now also RV3.1
- net at C6.2, C7.1, U2.1: now also D1.1 (K)
- net at D1.2 (A): now also RV3.2
- no-connect marks 0 -> 1
Changed lines of the file:
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@@
 	)
 	(junction
-		(at 148.59 102.87)
+		(at 152.4 39.37)
 		(diameter 0)
 		(color 0 0 0 0)
 	)
 	(junction
-		(at 152.4 39.37)
+		(at 128.27 125.73)
 		(diameter 0)
 		(color 0 0 0 0)
 	)
 	(junction
-		(at 128.27 125.73)
+		(at 148.59 102.87)
 		(diameter 0)
 		(color 0 0 0 0)
@@
 		(color 0 0 0 0)
 	)
+	(no_connect
+		(at 189.23 99.06)
+	)
 	(wire
 		(pts
@@
 	(wire
 		(pts
-			(xy 173.99 102.87) (xy 172.72 102.87)
-		)
-		(stroke
-			(width 0)
-			(type default)
-		)
-	)
-	(wire
-		(pts
 			(xy 137.16 142.24) (xy 153.67 142.24)
 		)
@@
 	(wire
 		(pts
-			(xy 152.4 40.64) (xy 152.4 39.37)
+			(xy 148.59 102.87) (xy 171.45 102.87)
 		)
 		(stroke
@@
 	(wire
 		(pts
-			(xy 68.58 116.84) (xy 96.52 116.84)
+			(xy 152.4 40.64) (xy 152.4 39.37)
 		)
 		(stroke
@@
 	(wire
 		(pts
-			(xy 43.18 116.84) (xy 48.26 116.84)
+			(xy 68.58 116.84) (xy 96.52 116.84)
 		)
 		(stroke
@@
 	(wire
 		(pts
-			(xy 148.59 102.87) (xy 165.1 102.87)
+			(xy 43.18 116.84) (xy 48.26 116.84)
 		)
 		(stroke
@@
 	(wire
 		(pts
+			(xy 189.23 106.68) (xy 199.39 106.68)
+		)
+		(stroke
+			(width 0)
+			(type default)
+		)
+	)
+	(wire
+		(pts
 			(xy 161.29 95.25) (xy 161.29 114.3)
 		)
@@
 	(wire
 		(pts
-			(xy 199.39 102.87) (xy 194.31 102.87)
+			(xy 199.39 77.47) (xy 215.9 77.47)
 		)
 		(stroke
@@
 	(wire
 		(pts
-			(xy 199.39 77.47) (xy 215.9 77.47)
+			(xy 96.52 102.87) (xy 114.3 102.87)
 		)
 		(stroke
@@
 	(wire
 		(pts
-			(xy 96.52 102.87) (xy 114.3 102.87)
+			(xy 129.54 102.87) (xy 137.16 102.87)
 		)
 		(stroke
@@
 	(wire
 		(pts
-			(xy 129.54 102.87) (xy 137.16 102.87)
+			(xy 179.07 102.87) (xy 185.42 102.87)
 		)
 		(stroke
@@
 	(wire
 		(pts
-			(xy 186.69 102.87) (xy 181.61 102.87)
-		)
-		(stroke
-			(width 0)
-			(type default)
-		)
-	)
-	(wire
-		(pts
 			(xy 137.16 95.25) (xy 137.16 96.52)
 		)
@@
 	(wire
 		(pts
-			(xy 199.39 77.47) (xy 199.39 102.87)
+			(xy 199.39 77.47) (xy 199.39 106.68)
 		)
 		(stroke
@@
 	)
 	(symbol
+		(lib_id "Diode:1N4148")
+		(at 175.26 102.87 0)
+		(unit 1)
+		(exclude_from_sim no)
+		(in_bom yes)
+		(on_board yes)
+		(dnp no)
+		(fields_autoplaced yes)
+		(property "Reference" "D1"
+			(at 175.26 96.52 0)
+			(effects
+				(font
+					(size 1.27 1.27)
+				)
+			)
+		)
+		(property "Value" "1N4148"
+			(at 175.26 99.06 0)
+			(effects
+				(font
+					(size 1.27 1.27)
+				)
+			)
+		)
+		(property "Footprint" "Diode_THT:D_DO-35_SOD27_P7.62mm_Horizontal"
+			(at 175.26 102.87 0)
+			(effects
+				(font
+					(size 1.27 1.27)
+				)
+				(hide yes)
+			)
+		)
+		(property "Datasheet" "https://assets.nexperia.com/documents/data-sheet/1N4148_1N4448.pdf"
+			(at 175.26 102.87 0)
+			(effects
+				(font
+					(size 1.27 1.27)
+				)
+				(hide yes)
+			)
+		)
+		(property "Description" "100V 0.15A standard switching diode, DO-35"
+			(at 175.26 102.87 0)
+			(effects
+				(font
+					(size 1.27 1.27)
+				)
+				(hide yes)
+			)
+		)
+		(property "Sim.Device" "D"
+			(at 175.26 102.87 0)
+			(effects
+				(font
+					(size 1.27 1.27)
+				)
+				(hide yes)
+			)
+		)
+		(property "Sim.Pins" "1=K 2=A"
+			(at 175.26 102.87 0)
+			(effects
+				(font
+					(size 1.27 1.27)
+				)
+				(hide yes)
+			)
+		)
+		(pin "1"
+		)
+		(pin "2"
+		)
+		(instances
+			(project ""
+				(path "/feb6dcc4-ba57-4640-ad64-1efd302ce012"
+					(reference "D1")
+					(unit 1)
+				)
+			)
+		)
+	)
+	(symbol
 		(lib_id "power:GND1")
 		(at 68.58 106.68 0)
@@
 	)
 	(symbol
-		(lib_id "Device:R_US")
-		(at 190.5 102.87 90)
-		(unit 1)
-		(exclude_from_sim no)
-		(in_bom yes)
-		(on_board yes)
-		(dnp no)
-		(fields_autoplaced yes)
-		(property "Reference" "R2"
-			(at 190.5 96.52 90)
-			(effects
-				(font
-					(size 1.27 1.27)
-				)
-			)
-		)
-		(property "Value" "1k ohm"
-			(at 190.5 99.06 90)
-			(effects
-				(font
-					(size 1.27 1.27)
-				)
-			)
-		)
-		(property "Footprint" ""
-			(at 190.754 101.854 90)
-			(effects
-				(font
-					(size 1.27 1.27)
-				)
-				(hide yes)
-			)
-		)
-		(property "Datasheet" "~"
-			(at 190.5 102.87 0)
-			(effects
-				(font
-					(size 1.27 1.27)
-				)
-				(hide yes)
-			)
-		)
-		(property "Description" "Resistor, US symbol"
-			(at 190.5 102.87 0)
-			(effects
-				(font
-					(size 1.27 1.27)
-				)
-				(hide yes)
-			)
-		)
-		(pin "1"
-		)
-		(pin "2"
-		)
-		(instances
-			(project ""
-				(path "/feb6dcc4-ba57-4640-ad64-1efd302ce012"
-					(reference "R2")
-					(unit 1)
-				)
-			)
-		)
-	)
-	(symbol
-		(lib_id "Device:LED")
-		(at 168.91 102.87 0)
-		(unit 1)
-		(exclude_from_sim no)
-		(in_bom yes)
-		(on_board yes)
-		(dnp no)
-		(fields_autoplaced yes)
-		(property "Reference" "D2"
-			(at 167.3225 96.52 0)
-			(effects
-				(font
-					(size 1.27 1.27)
-				)
-			)
-		)
-		(property "Value" "R_LED"
-			(at 167.3225 99.06 0)
-			(effects
-				(font
-					(size 1.27 1.27)
-				)
-			)
-		)
-		(property "Footprint" ""
-			(at 168.91 102.87 0)
-			(effects
-				(font
-					(size 1.27 1.27)
-				)
-				(hide yes)
-			)
-		)
-		(property "Datasheet" "~"
-			(at 168.91 102.87 0)
-			(effects
-				(font
-					(size 1.27 1.27)
-				)
-				(hide yes)
-			)
-		)
-		(property "Description" "Light emitting diode"
-			(at 168.91 102.87 0)
-			(effects
-				(font
-					(size 1.27 1.27)
-				)
-				(hide yes)
-			)
-		)
-		(property "Sim.Pins" "1=K 2=A"
-			(at 168.91 102.87 0)
-			(effects
-				(font
-					(size 1.27 1.27)
-				)
-				(hide yes)
-			)
-		)
-		(pin "2"
-		)
-		(pin "1"
-		)
-		(instances
-			(project ""
-				(path "/feb6dcc4-ba57-4640-ad64-1efd302ce012"
-					(reference "D2")
-					(unit 1)
-				)
-			)
-		)
-	)
-	(symbol
 		(lib_id "power:GND1")
 		(at 93.98 55.88 0)
@@
 	)
 	(symbol
-		(lib_id "Diode:1N4148")
-		(at 177.8 102.87 0)
+		(lib_id "Device:R_Potentiometer_US")
+		(at 189.23 102.87 180)
 		(unit 1)
 		(exclude_from_sim no)
@@
 		(on_board yes)
 		(dnp no)
-		(fields_autoplaced yes)
-		(property "Reference" "D1"
-			(at 177.8 96.52 0)
-			(effects
-				(font
-					(size 1.27 1.27)
-				)
-			)
-		)
-		(property "Value" "1N4148"
-			(at 177.8 99.06 0)
+		(property "Reference" "RV3"
+			(at 191.77 104.1401 0)
 			(effects
 				(font
 					(size 1.27 1.27)
 				)
+				(justify right)
 			)
 		)
-		(property "Footprint" "Diode_THT:D_DO-35_SOD27_P7.62mm_Horizontal"
-			(at 177.8 102.87 0)
+		(property "Value" "10k"
+			(at 191.77 101.6001 0)
 			(effects
 				(font
 					(size 1.27 1.27)
 				)
-				(hide yes)
+				(justify right)
 			)
 		)
-		(property "Datasheet" "https://assets.nexperia.com/documents/data-sheet/1N4148_1N4448.pdf"
-			(at 177.8 102.87 0)
+		(property "Footprint" ""
+			(at 189.23 102.87 0)
 			(effects
 				(font
@@
 			)
 		)
-		(property "Description" "100V 0.15A standard switching diode, DO-35"
-			(at 177.8 102.87 0)
+		(property "Datasheet" "~"
+			(at 189.23 102.87 0)
 			(effects
 				(font
@@
 			)
 		)
-		(property "Sim.Device" "D"
-			(at 177.8 102.87 0)
+		(property "Description" "Potentiometer, US symbol"
+			(at 189.23 102.87 0)
 			(effects
 				(font
@@
 			)
 		)
-		(property "Sim.Pins" "1=K 2=A"
-			(at 177.8 102.87 0)
-			(effects
-				(font
-					(size 1.27 1.27)
-				)
-				(hide yes)
-			)
+		(pin "3"
 		)
 		(pin "2"
@@
 		)
 		(instances
-			(project ""
+			(project "NodePilot"
 				(path "/feb6dcc4-ba57-4640-ad64-1efd302ce012"
-					(reference "D1")
+					(reference "RV3")
 					(unit 1)
 				)
